Commit message: Mapping now works without encoders

File: src/delivery_robot_description/urdf/accessories/rover_dev_payload.urdf (robot description, URDF)
Before this commit: robot rover_miti_payload, 1 links, 1 joints
Links:
- link payload_link: geometry collision mesh filename=file://$(find delivery_robot_description)/meshes/rover_payl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; visual mesh filename=file://$(find delivery_robot_description)/meshes/rover_payl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

File: src/delivery_robot_description/urdf/accessories/rplidar_s2.urdf (robot description, URDF)
Before this commit: robot rplidar_s2, 1 links, 1 joints
Links:
- link lidar_link: geometry collision mesh filename=file://$(find delivery_robot_description)/meshes/rplidar_s2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; visual mesh filename=file://$(find delivery_robot_description)/meshes/rplidar_s2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

File: src/delivery_robot_description/urdf/delivery_robot.urdf (robot description, URDF)
Before this commit: robot rover_4wd, 6 links, 5 joints
Links:
- link chassis_link: geometry collision mesh filename=file://$(find delivery_robot_description)/meshes/flipper_ch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; collision mesh filename=file://$(find delivery_robot_description)/meshes/flipper_tr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
- link fl_wheel_link: geometry collision mesh filename=file://$(find delivery_robot_description)/meshes/pro_tire.d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; visual mesh filename=file://$(find delivery_robot_description)/meshes/pro_tire.d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
- link fr_wheel_link: geometry collision mesh filename=file://$(find delivery_robot_description)/meshes/pro_tire.d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; visual mesh filename=file://$(find delivery_robot_description)/meshes/pro_tire.d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
- link rl_wheel_link: geometry collision mesh filename=file://$(find delivery_robot_description)/meshes/pro_tire.d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; visual mesh filename=file://$(find delivery_robot_description)/meshes/pro_tire.d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
- link rr_wheel_link: geometry collision mesh filename=file://$(find delivery_robot_description)/meshes/pro_tire.d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; visual mesh filename=file://$(find delivery_robot_description)/meshes/pro_tire.d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

File: src/delivery_robot_description/urdf/flipper.urdf (robot description, URDF)
Before this commit: robot rover_flipper, 8 links, 7 joints
Links:
- link bl_flipper_link: geometry collision mesh filename=file://$(find delivery_robot_description)/meshes/flipper.dae; visual mesh filename=file://$(find delivery_robot_description)/meshes/flipper.dae
- link br_flipper_link: geometry collision mesh filename=file://$(find delivery_robot_description)/meshes/flipper.dae; visual mesh filename=file://$(find delivery_robot_description)/meshes/flipper.dae
- link chassis_link: geometry collision mesh filename=file://$(find delivery_robot_description)/meshes/flipper_ch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; visual mesh filename=file://$(find delivery_robot_description)/meshes/flipper_ch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
- link fl_flipper_link: geometry collision mesh filename=file://$(find delivery_robot_description)/meshes/flipper.dae; visual mesh filename=file://$(find delivery_robot_description)/meshes/flipper.dae
- link fr_flipper_link: geometry collision mesh filename=file://$(find delivery_robot_description)/meshes/flipper.dae; visual mesh filename=file://$(find delivery_robot_description)/meshes/flipper.dae
- link left_track_link: geometry collision mesh filename=file://$(find delivery_robot_description)/meshes/flipper_tr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; visual mesh filename=file://$(find delivery_robot_description)/meshes/flipper_tr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
- link right_track_link: geometry collision mesh filename=file://$(find delivery_robot_description)/meshes/flipper_tr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; visual mesh filename=file://$(find delivery_robot_description)/meshes/flipper_tr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

File: src/delivery_robot_description/urdf/max.urdf (robot description, URDF)
Before this commit: robot rover_miti, 6 links, 5 joints
Links:
- link chassis_link: geometry collision mesh filename=file://$(find delivery_robot_description)/meshes/max_chassi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; visual mesh filename=file://$(find delivery_robot_description)/meshes/max_chassi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
- link fl_wheel_link: geometry collision mesh filename=file://$(find delivery_robot_description)/meshes/max_wheels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; visual mesh filename=file://$(find delivery_robot_description)/meshes/max_wheels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
- link fr_wheel_link: geometry collision mesh filename=file://$(find delivery_robot_description)/meshes/max_wheels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; visual mesh filename=file://$(find delivery_robot_description)/meshes/max_wheels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
- link rl_wheel_link: geometry collision mesh filename=file://$(find delivery_robot_description)/meshes/max_wheels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; visual mesh filename=file://$(find delivery_robot_description)/meshes/max_wheels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
- link rr_wheel_link: geometry collision mesh filename=file://$(find delivery_robot_description)/meshes/max_wheels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; visual mesh filename=file://$(find delivery_robot_description)/meshes/max_wheels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

File: src/delivery_robot_description/urdf/max_100.urdf (robot description, URDF)
Before this commit: robot rover_max, 6 links, 5 joints
Links:
- link chassis_link: geometry collision mesh filename=file://$(find delivery_robot_description)/meshes/max_chassi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; visual mesh filename=file://$(find delivery_robot_description)/meshes/max_chassi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
- link fl_wheel_link: geometry collision mesh filename=file://$(find delivery_robot_description)/meshes/max_wheels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; visual mesh filename=file://$(find delivery_robot_description)/meshes/max_wheels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
- link fr_wheel_link: geometry collision mesh filename=file://$(find delivery_robot_description)/meshes/max_wheels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; visual mesh filename=file://$(find delivery_robot_description)/meshes/max_wheels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
- link rl_wheel_link: geometry collision mesh filename=file://$(find delivery_robot_description)/meshes/max_wheels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; visual mesh filename=file://$(find delivery_robot_description)/meshes/max_wheels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
- link rr_wheel_link: geometry collision mesh filename=file://$(find delivery_robot_description)/meshes/max_wheels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; visual mesh filename=file://$(find delivery_robot_description)/meshes/max_wheels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

File: src/delivery_robot_description/urdf/max_100_neo.urdf (robot description, URDF)
Before this commit: robot rover_max, 6 links, 5 joints
Links:
- link chassis_link: geometry collision mesh filename=file://$(find delivery_robot_description)/meshes/max_chassi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; visual mesh filename=file://$(find delivery_robot_description)/meshes/max_chassi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
- link fl_wheel_link: geometry collision mesh filename=file://$(find delivery_robot_description)/meshes/max_wheels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; visual mesh filename=file://$(find delivery_robot_description)/meshes/max_wheels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
- link fr_wheel_link: geometry collision mesh filename=file://$(find delivery_robot_description)/meshes/max_wheels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; visual mesh filename=file://$(find delivery_robot_description)/meshes/max_wheels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
- link rl_wheel_link: geometry collision mesh filename=file://$(find delivery_robot_description)/meshes/max_wheels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; visual mesh filename=file://$(find delivery_robot_description)/meshes/max_wheels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
- link rr_wheel_link: geometry collision mesh filename=file://$(find delivery_robot_description)/meshes/max_wheels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; visual mesh filename=file://$(find delivery_robot_description)/meshes/max_wheels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

File: src/delivery_robot_description/urdf/max_130.urdf (robot description, URDF)
Before this commit: robot rover_max, 6 links, 5 joints
Links:
- link chassis_link: geometry collision mesh filename=file://$(find delivery_robot_description)/meshes/max_chassi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; visual mesh filename=file://$(find delivery_robot_description)/meshes/max_chassi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
- link fl_wheel_link: geometry collision mesh filename=file://$(find delivery_robot_description)/meshes/max_wheels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; visual mesh filename=file://$(find delivery_robot_description)/meshes/max_wheels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
- link fr_wheel_link: geometry collision mesh filename=file://$(find delivery_robot_description)/meshes/max_wheels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; visual mesh filename=file://$(find delivery_robot_description)/meshes/max_wheels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
- link rl_wheel_link: geometry collision mesh filename=file://$(find delivery_robot_description)/meshes/max_wheels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; visual mesh filename=file://$(find delivery_robot_description)/meshes/max_wheels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
- link rr_wheel_link: geometry collision mesh filename=file://$(find delivery_robot_description)/meshes/max_wheels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; visual mesh filename=file://$(find delivery_robot_description)/meshes/max_wheels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

File: src/delivery_robot_description/urdf/max_130_neo.urdf (robot description, URDF)
Before this commit: robot rover_max, 6 links, 5 joints
Links:
- link chassis_link: geometry collision mesh filename=file://$(find delivery_robot_description)/meshes/max_chassi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; visual mesh filename=file://$(find delivery_robot_description)/meshes/max_chassi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
- link fl_wheel_link: geometry collision mesh filename=file://$(find delivery_robot_description)/meshes/max_wheels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; visual mesh filename=file://$(find delivery_robot_description)/meshes/max_wheels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
- link fr_wheel_link: geometry collision mesh filename=file://$(find delivery_robot_description)/meshes/max_wheels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; visual mesh filename=file://$(find delivery_robot_description)/meshes/max_wheels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
- link rl_wheel_link: geometry collision mesh filename=file://$(find delivery_robot_description)/meshes/max_wheels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; visual mesh filename=file://$(find delivery_robot_description)/meshes/max_wheels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
- link rr_wheel_link: geometry collision mesh filename=file://$(find delivery_robot_description)/meshes/max_wheels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; visual mesh filename=file://$(find delivery_robot_description)/meshes/max_wheels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

File: src/delivery_robot_description/urdf/max_150.urdf (robot description, URDF)
Before this commit: robot rover_max, 6 links, 5 joints
Links:
- link chassis_link: geometry collision mesh filename=file://$(find delivery_robot_description)/meshes/max_chassi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; visual mesh filename=file://$(find delivery_robot_description)/meshes/max_chassi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
- link fl_wheel_link: geometry collision mesh filename=file://$(find delivery_robot_description)/meshes/max_wheels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; visual mesh filename=file://$(find delivery_robot_description)/meshes/max_wheels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
- link fr_wheel_link: geometry collision mesh filename=file://$(find delivery_robot_description)/meshes/max_wheels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; visual mesh filename=file://$(find delivery_robot_description)/meshes/max_wheels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
- link rl_wheel_link: geometry collision mesh filename=file://$(find delivery_robot_description)/meshes/max_wheels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; visual mesh filename=file://$(find delivery_robot_description)/meshes/max_wheels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
- link rr_wheel_link: geometry collision mesh filename=file://$(find delivery_robot_description)/meshes/max_wheels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; visual mesh filename=file://$(find delivery_robot_description)/meshes/max_wheels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

File: src/delivery_robot_description/urdf/max_150_neo.urdf (robot description, URDF)
Before this commit: robot rover_max, 6 links, 5 joints
Links:
- link chassis_link: geometry collision mesh filename=file://$(find delivery_robot_description)/meshes/max_chassi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; visual mesh filename=file://$(find delivery_robot_description)/meshes/max_chassi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
- link fl_wheel_link: geometry collision mesh filename=file://$(find delivery_robot_description)/meshes/max_wheels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; visual mesh filename=file://$(find delivery_robot_description)/meshes/max_wheels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
- link fr_wheel_link: geometry collision mesh filename=file://$(find delivery_robot_description)/meshes/max_wheels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; visual mesh filename=file://$(find delivery_robot_description)/meshes/max_wheels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
- link rl_wheel_link: geometry collision mesh filename=file://$(find delivery_robot_description)/meshes/max_wheels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; visual mesh filename=file://$(find delivery_robot_description)/meshes/max_wheels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
- link rr_wheel_link: geometry collision mesh filename=file://$(find delivery_robot_description)/meshes/max_wheels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; visual mesh filename=file://$(find delivery_robot_description)/meshes/max_wheels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

File: src/delivery_robot_description/urdf/max_65.urdf (robot description, URDF)
Before this commit: robot rover_max, 6 links, 5 joints
Links:
- link chassis_link: geometry collision mesh filename=file://$(find delivery_robot_description)/meshes/max_chassi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; visual mesh filename=file://$(find delivery_robot_description)/meshes/max_chassi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
- link fl_wheel_link: geometry collision mesh filename=file://$(find delivery_robot_description)/meshes/65wheels.d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; visual mesh filename=file://$(find delivery_robot_description)/meshes/65wheels.d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
- link fr_wheel_link: geometry collision mesh filename=file://$(find delivery_robot_description)/meshes/65wheels.d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; visual mesh filename=file://$(find delivery_robot_description)/meshes/65wheels.d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
- link rl_wheel_link: geometry collision mesh filename=file://$(find delivery_robot_description)/meshes/65wheels.d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; visual mesh filename=file://$(find delivery_robot_description)/meshes/65wheels.d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
- link rr_wheel_link: geometry collision mesh filename=file://$(find delivery_robot_description)/meshes/65wheels.d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; visual mesh filename=file://$(find delivery_robot_description)/meshes/65wheels.d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

File: src/delivery_robot_description/urdf/mega.urdf (robot description, URDF)
Before this commit: robot rover_mega, 6 links, 5 joints
Links:
- link chassis_link: geometry collision mesh filename=file://$(find delivery_robot_description)/meshes/mega_chass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; visual mesh filename=file://$(find delivery_robot_description)/meshes/mega_chass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
- link fl_wheel_link: geometry collision mesh filename=file://$(find delivery_robot_description)/meshes/mega_wheel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; visual mesh filename=file://$(find delivery_robot_description)/meshes/mega_wheel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
- link fr_wheel_link: geometry collision mesh filename=file://$(find delivery_robot_description)/meshes/mega_wheel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; visual mesh filename=file://$(find delivery_robot_description)/meshes/mega_wheel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
- link rl_wheel_link: geometry collision mesh filename=file://$(find delivery_robot_description)/meshes/mega_wheel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; visual mesh filename=file://$(find delivery_robot_description)/meshes/mega_wheel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
- link rr_wheel_link: geometry collision mesh filename=file://$(find delivery_robot_description)/meshes/mega_wheel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; visual mesh filename=file://$(find delivery_robot_description)/meshes/mega_wheel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

File: src/delivery_robot_description/urdf/mini.urdf (robot description, URDF)
Before this commit: robot rover_mini, 6 links, 5 joints
Links:
- link chassis_link: geometry collision mesh filename=file://$(find delivery_robot_description)/meshes/mini_chass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; visual mesh filename=file://$(find delivery_robot_description)/meshes/mini_chass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
- link fl_wheel_link: geometry collision mesh filename=file://$(find delivery_robot_description)/meshes/65wheels.d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; visual mesh filename=file://$(find delivery_robot_description)/meshes/65wheels.d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
- link fr_wheel_link: geometry collision mesh filename=file://$(find delivery_robot_description)/meshes/65wheels.d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; visual mesh filename=file://$(find delivery_robot_description)/meshes/65wheels.d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
- link rl_wheel_link: geometry collision mesh filename=file://$(find delivery_robot_description)/meshes/65wheels.d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; visual mesh filename=file://$(find delivery_robot_description)/meshes/65wheels.d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
- link rr_wheel_link: geometry collision mesh filename=file://$(find delivery_robot_description)/meshes/65wheels.d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; visual mesh filename=file://$(find delivery_robot_description)/meshes/65wheels.d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

File: src/delivery_robot_description/urdf/miti.urdf (robot description, URDF)
Before this commit: robot rover_miti, 6 links, 5 joints
Links:
- link chassis_link: geometry collision mesh filename=file://$(find delivery_robot_description)/meshes/miti_chass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; visual mesh filename=file://$(find delivery_robot_description)/meshes/miti_chass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
- link fl_wheel_link: geometry collision mesh filename=file://$(find delivery_robot_description)/meshes/hub_10in.d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; visual mesh filename=file://$(find delivery_robot_description)/meshes/hub_10in.d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
- link fr_wheel_link: geometry collision mesh filename=file://$(find delivery_robot_description)/meshes/hub_10in.d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; visual mesh filename=file://$(find delivery_robot_description)/meshes/hub_10in.d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
- link rl_wheel_link: geometry collision mesh filename=file://$(find delivery_robot_description)/meshes/hub_10in.d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; visual mesh filename=file://$(find delivery_robot_description)/meshes/hub_10in.d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
- link rr_wheel_link: geometry collision mesh filename=file://$(find delivery_robot_description)/meshes/hub_10in.d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; visual mesh filename=file://$(find delivery_robot_description)/meshes/hub_10in.d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

File: src/delivery_robot_description/urdf/miti_65.urdf (robot description, URDF)
Before this commit: robot rover_miti, 6 links, 5 joints
Links:
- link chassis_link: geometry collision mesh filename=file://$(find delivery_robot_description)/meshes/miti_chass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; visual mesh filename=file://$(find delivery_robot_description)/meshes/miti_chass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
- link fl_wheel_link: geometry collision mesh filename=file://$(find delivery_robot_description)/meshes/65wheels.d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; visual mesh filename=file://$(find delivery_robot_description)/meshes/65wheels.d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
- link fr_wheel_link: geometry collision mesh filename=file://$(find delivery_robot_description)/meshes/65wheels.d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; visual mesh filename=file://$(find delivery_robot_description)/meshes/65wheels.d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
- link rl_wheel_link: geometry collision mesh filename=file://$(find delivery_robot_description)/meshes/65wheels.d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; visual mesh filename=file://$(find delivery_robot_description)/meshes/65wheels.d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
- link rr_wheel_link: geometry collision mesh filename=file://$(find delivery_robot_description)/meshes/65wheels.d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; visual mesh filename=file://$(find delivery_robot_description)/meshes/65wheels.d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

File: src/delivery_robot_description/urdf/rover_2wd.urdf (robot description, URDF)
Before this commit: robot rover_2wd, 8 links, 7 joints
Links:
- link chassis_link: geometry collision mesh filename=file://$(find delivery_robot_description)/meshes/rover_2wd_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; visual mesh filename=file://$(find delivery_robot_description)/meshes/rover_2wd_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
- link fl_wheel_link: geometry collision mesh filename=file://$(find delivery_robot_description)/meshes/pro_tire.d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; visual mesh filename=file://$(find delivery_robot_description)/meshes/pro_tire.d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
- link fr_wheel_link: geometry collision mesh filename=file://$(find delivery_robot_description)/meshes/pro_tire.d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; visual mesh filename=file://$(find delivery_robot_description)/meshes/pro_tire.d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
- link rl_castor_housing_link: geometry collision mesh filename=file://$(find delivery_robot_description)/meshes/castor_hou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; visual mesh filename=file://$(find delivery_robot_description)/meshes/castor_hou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
- link rl_castor_link: geometry collision mesh filename=file://$(find delivery_robot_description)/meshes/castor.dae; visual mesh filename=file://$(find delivery_robot_description)/meshes/castor.dae
- link rr_castor_housing_link: geometry collision mesh filename=file://$(find delivery_robot_description)/meshes/castor_hou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; visual mesh filename=file://$(find delivery_robot_description)/meshes/castor_hou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
- link rr_castor_link: geometry collision mesh filename=file://$(find delivery_robot_description)/meshes/castor.dae; visual mesh filename=file://$(find delivery_robot_description)/meshes/castor.dae
