Commit message: Removed description packaged because it was not used

File: src/delivery_robot_bringup/urdf/accessories/rover_dev_payload.urdf (robot description, URDF)
Before this commit: robot rover_miti_payload, 1 links, 1 joints
Links:
- link payload_link: geometry collision mesh filename=file://$(find delivery_robot_bringup)/meshes/rover_payload.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; visual mesh filename=file://$(find delivery_robot_bringup)/meshes/rover_payload.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

File: src/delivery_robot_bringup/urdf/accessories/rplidar_s2.urdf (robot description, URDF)
Before this commit: robot rplidar_s2, 1 links, 1 joints
Links:
- link lidar_link: geometry collision mesh filename=file://$(find delivery_robot_bringup)/meshes/rplidar_s2.dae; visual mesh filename=file://$(find delivery_robot_bringup)/meshes/rplidar_s2.dae

File: src/delivery_robot_bringup/urdf/delivery_robot.urdf (robot description, URDF)
Before this commit: robot rover_4wd, 6 links, 5 joints
Links:
- link chassis_link: geometry collision mesh filename=file://$(find delivery_robot_bringup)/meshes/flipper_chassi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; collision mesh filename=file://$(find delivery_robot_bringup)/meshes/flipper_track.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
- link fl_wheel_link: geometry collision mesh filename=file://$(find delivery_robot_bringup)/meshes/pro_tire.dae; visual mesh filename=file://$(find delivery_robot_bringup)/meshes/pro_tire.dae
- link fr_wheel_link: geometry collision mesh filename=file://$(find delivery_robot_bringup)/meshes/pro_tire.dae; visual mesh filename=file://$(find delivery_robot_bringup)/meshes/pro_tire.dae
- link rl_wheel_link: geometry collision mesh filename=file://$(find delivery_robot_bringup)/meshes/pro_tire.dae; visual mesh filename=file://$(find delivery_robot_bringup)/meshes/pro_tire.dae
- link rr_wheel_link: geometry collision mesh filename=file://$(find delivery_robot_bringup)/meshes/pro_tire.dae; visual mesh filename=file://$(find delivery_robot_bringup)/meshes/pro_tire.dae

File: src/delivery_robot_bringup/urdf/flipper.urdf (robot description, URDF)
Before this commit: robot rover_flipper, 8 links, 7 joints
Links:
- link bl_flipper_link: geometry collision mesh filename=file://$(find delivery_robot_bringup)/meshes/flipper.dae; visual mesh filename=file://$(find delivery_robot_bringup)/meshes/flipper.dae
- link br_flipper_link: geometry collision mesh filename=file://$(find delivery_robot_bringup)/meshes/flipper.dae; visual mesh filename=file://$(find delivery_robot_bringup)/meshes/flipper.dae
- link chassis_link: geometry collision mesh filename=file://$(find delivery_robot_bringup)/meshes/flipper_chassi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; visual mesh filename=file://$(find delivery_robot_bringup)/meshes/flipper_chassi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
- link fl_flipper_link: geometry collision mesh filename=file://$(find delivery_robot_bringup)/meshes/flipper.dae; visual mesh filename=file://$(find delivery_robot_bringup)/meshes/flipper.dae
- link fr_flipper_link: geometry collision mesh filename=file://$(find delivery_robot_bringup)/meshes/flipper.dae; visual mesh filename=file://$(find delivery_robot_bringup)/meshes/flipper.dae
- link left_track_link: geometry collision mesh filename=file://$(find delivery_robot_bringup)/meshes/flipper_track.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; visual mesh filename=file://$(find delivery_robot_bringup)/meshes/flipper_track.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
- link right_track_link: geometry collision mesh filename=file://$(find delivery_robot_bringup)/meshes/flipper_track.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; visual mesh filename=file://$(find delivery_robot_bringup)/meshes/flipper_track.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

File: src/delivery_robot_bringup/urdf/max.urdf (robot description, URDF)
Before this commit: robot rover_miti, 6 links, 5 joints
Links:
- link chassis_link: geometry collision mesh filename=file://$(find delivery_robot_bringup)/meshes/max_chassis.dae; visual mesh filename=file://$(find delivery_robot_bringup)/meshes/max_chassis.dae
- link fl_wheel_link: geometry collision mesh filename=file://$(find delivery_robot_bringup)/meshes/max_wheels.dae; visual mesh filename=file://$(find delivery_robot_bringup)/meshes/max_wheels.dae
- link fr_wheel_link: geometry collision mesh filename=file://$(find delivery_robot_bringup)/meshes/max_wheels.dae; visual mesh filename=file://$(find delivery_robot_bringup)/meshes/max_wheels.dae
- link rl_wheel_link: geometry collision mesh filename=file://$(find delivery_robot_bringup)/meshes/max_wheels.dae; visual mesh filename=file://$(find delivery_robot_bringup)/meshes/max_wheels.dae
- link rr_wheel_link: geometry collision mesh filename=file://$(find delivery_robot_bringup)/meshes/max_wheels.dae; visual mesh filename=file://$(find delivery_robot_bringup)/meshes/max_wheels.dae

File: src/delivery_robot_bringup/urdf/max_100.urdf (robot description, URDF)
Before this commit: robot rover_max, 6 links, 5 joints
Links:
- link chassis_link: geometry collision mesh filename=file://$(find delivery_robot_bringup)/meshes/max_chassis.dae; visual mesh filename=file://$(find delivery_robot_bringup)/meshes/max_chassis.dae
- link fl_wheel_link: geometry collision mesh filename=file://$(find delivery_robot_bringup)/meshes/max_wheels_10i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; visual mesh filename=file://$(find delivery_robot_bringup)/meshes/max_wheels_10i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
- link fr_wheel_link: geometry collision mesh filename=file://$(find delivery_robot_bringup)/meshes/max_wheels_10i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; visual mesh filename=file://$(find delivery_robot_bringup)/meshes/max_wheels_10i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
- link rl_wheel_link: geometry collision mesh filename=file://$(find delivery_robot_bringup)/meshes/max_wheels_10i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; visual mesh filename=file://$(find delivery_robot_bringup)/meshes/max_wheels_10i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
- link rr_wheel_link: geometry collision mesh filename=file://$(find delivery_robot_bringup)/meshes/max_wheels_10i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; visual mesh filename=file://$(find delivery_robot_bringup)/meshes/max_wheels_10i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

File: src/delivery_robot_bringup/urdf/max_100_neo.urdf (robot description, URDF)
Before this commit: robot rover_max, 6 links, 5 joints
Links:
- link chassis_link: geometry collision mesh filename=file://$(find delivery_robot_bringup)/meshes/max_chassis_ne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; visual mesh filename=file://$(find delivery_robot_bringup)/meshes/max_chassis_ne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
- link fl_wheel_link: geometry collision mesh filename=file://$(find delivery_robot_bringup)/meshes/max_wheels_10i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; visual mesh filename=file://$(find delivery_robot_bringup)/meshes/max_wheels_10i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
- link fr_wheel_link: geometry collision mesh filename=file://$(find delivery_robot_bringup)/meshes/max_wheels_10i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; visual mesh filename=file://$(find delivery_robot_bringup)/meshes/max_wheels_10i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
- link rl_wheel_link: geometry collision mesh filename=file://$(find delivery_robot_bringup)/meshes/max_wheels_10i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; visual mesh filename=file://$(find delivery_robot_bringup)/meshes/max_wheels_10i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
- link rr_wheel_link: geometry collision mesh filename=file://$(find delivery_robot_bringup)/meshes/max_wheels_10i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; visual mesh filename=file://$(find delivery_robot_bringup)/meshes/max_wheels_10i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

File: src/delivery_robot_bringup/urdf/max_130.urdf (robot description, URDF)
Before this commit: robot rover_max, 6 links, 5 joints
Links:
- link chassis_link: geometry collision mesh filename=file://$(find delivery_robot_bringup)/meshes/max_chassis.dae; visual mesh filename=file://$(find delivery_robot_bringup)/meshes/max_chassis.dae
- link fl_wheel_link: geometry collision mesh filename=file://$(find delivery_robot_bringup)/meshes/max_wheels_13i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; visual mesh filename=file://$(find delivery_robot_bringup)/meshes/max_wheels_13i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
- link fr_wheel_link: geometry collision mesh filename=file://$(find delivery_robot_bringup)/meshes/max_wheels_13i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; visual mesh filename=file://$(find delivery_robot_bringup)/meshes/max_wheels_13i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
- link rl_wheel_link: geometry collision mesh filename=file://$(find delivery_robot_bringup)/meshes/max_wheels_13i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; visual mesh filename=file://$(find delivery_robot_bringup)/meshes/max_wheels_13i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
- link rr_wheel_link: geometry collision mesh filename=file://$(find delivery_robot_bringup)/meshes/max_wheels_13i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; visual mesh filename=file://$(find delivery_robot_bringup)/meshes/max_wheels_13i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

File: src/delivery_robot_bringup/urdf/max_130_neo.urdf (robot description, URDF)
Before this commit: robot rover_max, 6 links, 5 joints
Links:
- link chassis_link: geometry collision mesh filename=file://$(find delivery_robot_bringup)/meshes/max_chassis_ne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; visual mesh filename=file://$(find delivery_robot_bringup)/meshes/max_chassis_ne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
- link fl_wheel_link: geometry collision mesh filename=file://$(find delivery_robot_bringup)/meshes/max_wheels_13i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; visual mesh filename=file://$(find delivery_robot_bringup)/meshes/max_wheels_13i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
- link fr_wheel_link: geometry collision mesh filename=file://$(find delivery_robot_bringup)/meshes/max_wheels_13i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; visual mesh filename=file://$(find delivery_robot_bringup)/meshes/max_wheels_13i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
- link rl_wheel_link: geometry collision mesh filename=file://$(find delivery_robot_bringup)/meshes/max_wheels_13i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; visual mesh filename=file://$(find delivery_robot_bringup)/meshes/max_wheels_13i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
- link rr_wheel_link: geometry collision mesh filename=file://$(find delivery_robot_bringup)/meshes/max_wheels_13i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; visual mesh filename=file://$(find delivery_robot_bringup)/meshes/max_wheels_13i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

File: src/delivery_robot_bringup/urdf/max_150.urdf (robot description, URDF)
Before this commit: robot rover_max, 6 links, 5 joints
Links:
- link chassis_link: geometry collision mesh filename=file://$(find delivery_robot_bringup)/meshes/max_chassis.dae; visual mesh filename=file://$(find delivery_robot_bringup)/meshes/max_chassis.dae
- link fl_wheel_link: geometry collision mesh filename=file://$(find delivery_robot_bringup)/meshes/max_wheels_15i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; visual mesh filename=file://$(find delivery_robot_bringup)/meshes/max_wheels_15i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
- link fr_wheel_link: geometry collision mesh filename=file://$(find delivery_robot_bringup)/meshes/max_wheels_15i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; visual mesh filename=file://$(find delivery_robot_bringup)/meshes/max_wheels_15i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
- link rl_wheel_link: geometry collision mesh filename=file://$(find delivery_robot_bringup)/meshes/max_wheels_15i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; visual mesh filename=file://$(find delivery_robot_bringup)/meshes/max_wheels_15i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
- link rr_wheel_link: geometry collision mesh filename=file://$(find delivery_robot_bringup)/meshes/max_wheels_15i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; visual mesh filename=file://$(find delivery_robot_bringup)/meshes/max_wheels_15i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

File: src/delivery_robot_bringup/urdf/max_150_neo.urdf (robot description, URDF)
Before this commit: robot rover_max, 6 links, 5 joints
Links:
- link chassis_link: geometry collision mesh filename=file://$(find delivery_robot_bringup)/meshes/max_chassis_ne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; visual mesh filename=file://$(find delivery_robot_bringup)/meshes/max_chassis_ne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
- link fl_wheel_link: geometry collision mesh filename=file://$(find delivery_robot_bringup)/meshes/max_wheels_15i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; visual mesh filename=file://$(find delivery_robot_bringup)/meshes/max_wheels_15i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
- link fr_wheel_link: geometry collision mesh filename=file://$(find delivery_robot_bringup)/meshes/max_wheels_15i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; visual mesh filename=file://$(find delivery_robot_bringup)/meshes/max_wheels_15i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
- link rl_wheel_link: geometry collision mesh filename=file://$(find delivery_robot_bringup)/meshes/max_wheels_15i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; visual mesh filename=file://$(find delivery_robot_bringup)/meshes/max_wheels_15i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
- link rr_wheel_link: geometry collision mesh filename=file://$(find delivery_robot_bringup)/meshes/max_wheels_15i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; visual mesh filename=file://$(find delivery_robot_bringup)/meshes/max_wheels_15i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

File: src/delivery_robot_bringup/urdf/max_65.urdf (robot description, URDF)
Before this commit: robot rover_max, 6 links, 5 joints
Links:
- link chassis_link: geometry collision mesh filename=file://$(find delivery_robot_bringup)/meshes/max_chassis.dae; visual mesh filename=file://$(find delivery_robot_bringup)/meshes/max_chassis.dae
- link fl_wheel_link: geometry collision mesh filename=file://$(find delivery_robot_bringup)/meshes/65wheels.dae; visual mesh filename=file://$(find delivery_robot_bringup)/meshes/65wheels.dae
- link fr_wheel_link: geometry collision mesh filename=file://$(find delivery_robot_bringup)/meshes/65wheels.dae; visual mesh filename=file://$(find delivery_robot_bringup)/meshes/65wheels.dae
- link rl_wheel_link: geometry collision mesh filename=file://$(find delivery_robot_bringup)/meshes/65wheels.dae; visual mesh filename=file://$(find delivery_robot_bringup)/meshes/65wheels.dae
- link rr_wheel_link: geometry collision mesh filename=file://$(find delivery_robot_bringup)/meshes/65wheels.dae; visual mesh filename=file://$(find delivery_robot_bringup)/meshes/65wheels.dae

File: src/delivery_robot_bringup/urdf/mega.urdf (robot description, URDF)
Before this commit: robot rover_mega, 6 links, 5 joints
Links:
- link chassis_link: geometry collision mesh filename=file://$(find delivery_robot_bringup)/meshes/mega_chassis.d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; visual mesh filename=file://$(find delivery_robot_bringup)/meshes/mega_chassis.d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
- link fl_wheel_link: geometry collision mesh filename=file://$(find delivery_robot_bringup)/meshes/mega_wheels.dae; visual mesh filename=file://$(find delivery_robot_bringup)/meshes/mega_wheels.dae
- link fr_wheel_link: geometry collision mesh filename=file://$(find delivery_robot_bringup)/meshes/mega_wheels.dae; visual mesh filename=file://$(find delivery_robot_bringup)/meshes/mega_wheels.dae
- link rl_wheel_link: geometry collision mesh filename=file://$(find delivery_robot_bringup)/meshes/mega_wheels.dae; visual mesh filename=file://$(find delivery_robot_bringup)/meshes/mega_wheels.dae
- link rr_wheel_link: geometry collision mesh filename=file://$(find delivery_robot_bringup)/meshes/mega_wheels.dae; visual mesh filename=file://$(find delivery_robot_bringup)/meshes/mega_wheels.dae

File: src/delivery_robot_bringup/urdf/mini.urdf (robot description, URDF)
Before this commit: robot rover_mini, 6 links, 5 joints
Links:
- link chassis_link: geometry collision mesh filename=file://$(find delivery_robot_bringup)/meshes/mini_chassis_n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; visual mesh filename=file://$(find delivery_robot_bringup)/meshes/mini_chassis_n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
- link fl_wheel_link: geometry collision mesh filename=file://$(find delivery_robot_bringup)/meshes/65wheels.dae; visual mesh filename=file://$(find delivery_robot_bringup)/meshes/65wheels.dae
- link fr_wheel_link: geometry collision mesh filename=file://$(find delivery_robot_bringup)/meshes/65wheels.dae; visual mesh filename=file://$(find delivery_robot_bringup)/meshes/65wheels.dae
- link rl_wheel_link: geometry collision mesh filename=file://$(find delivery_robot_bringup)/meshes/65wheels.dae; visual mesh filename=file://$(find delivery_robot_bringup)/meshes/65wheels.dae
- link rr_wheel_link: geometry collision mesh filename=file://$(find delivery_robot_bringup)/meshes/65wheels.dae; visual mesh filename=file://$(find delivery_robot_bringup)/meshes/65wheels.dae

File: src/delivery_robot_bringup/urdf/miti.urdf (robot description, URDF)
Before this commit: robot rover_miti, 6 links, 5 joints
Links:
- link chassis_link: geometry collision mesh filename=file://$(find delivery_robot_bringup)/meshes/miti_chassis_n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; visual mesh filename=file://$(find delivery_robot_bringup)/meshes/miti_chassis_n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
- link fl_wheel_link: geometry collision mesh filename=file://$(find delivery_robot_bringup)/meshes/hub_10in.dae; visual mesh filename=file://$(find delivery_robot_bringup)/meshes/hub_10in.dae
- link fr_wheel_link: geometry collision mesh filename=file://$(find delivery_robot_bringup)/meshes/hub_10in.dae; visual mesh filename=file://$(find delivery_robot_bringup)/meshes/hub_10in.dae
- link rl_wheel_link: geometry collision mesh filename=file://$(find delivery_robot_bringup)/meshes/hub_10in.dae; visual mesh filename=file://$(find delivery_robot_bringup)/meshes/hub_10in.dae
- link rr_wheel_link: geometry collision mesh filename=file://$(find delivery_robot_bringup)/meshes/hub_10in.dae; visual mesh filename=file://$(find delivery_robot_bringup)/meshes/hub_10in.dae

File: src/delivery_robot_bringup/urdf/miti_65.urdf (robot description, URDF)
Before this commit: robot rover_miti, 6 links, 5 joints
Links:
- link chassis_link: geometry collision mesh filename=file://$(find delivery_robot_bringup)/meshes/miti_chassis_n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; visual mesh filename=file://$(find delivery_robot_bringup)/meshes/miti_chassis_n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
- link fl_wheel_link: geometry collision mesh filename=file://$(find delivery_robot_bringup)/meshes/65wheels.dae; visual mesh filename=file://$(find delivery_robot_bringup)/meshes/65wheels.dae
- link fr_wheel_link: geometry collision mesh filename=file://$(find delivery_robot_bringup)/meshes/65wheels.dae; visual mesh filename=file://$(find delivery_robot_bringup)/meshes/65wheels.dae
- link rl_wheel_link: geometry collision mesh filename=file://$(find delivery_robot_bringup)/meshes/65wheels.dae; visual mesh filename=file://$(find delivery_robot_bringup)/meshes/65wheels.dae
- link rr_wheel_link: geometry collision mesh filename=file://$(find delivery_robot_bringup)/meshes/65wheels.dae; visual mesh filename=file://$(find delivery_robot_bringup)/meshes/65wheels.dae

File: src/delivery_robot_bringup/urdf/rover_2wd.urdf (robot description, URDF)
Before this commit: robot rover_2wd, 8 links, 7 joints
Links:
- link chassis_link: geometry collision mesh filename=file://$(find delivery_robot_bringup)/meshes/rover_2wd_core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; visual mesh filename=file://$(find delivery_robot_bringup)/meshes/rover_2wd_core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
- link fl_wheel_link: geometry collision mesh filename=file://$(find delivery_robot_bringup)/meshes/pro_tire.dae; visual mesh filename=file://$(find delivery_robot_bringup)/meshes/pro_tire.dae
- link fr_wheel_link: geometry collision mesh filename=file://$(find delivery_robot_bringup)/meshes/pro_tire.dae; visual mesh filename=file://$(find delivery_robot_bringup)/meshes/pro_tire.dae
- link rl_castor_housing_link: geometry collision mesh filename=file://$(find delivery_robot_bringup)/meshes/castor_housing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; visual mesh filename=file://$(find delivery_robot_bringup)/meshes/castor_housing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
- link rl_castor_link: geometry collision mesh filename=file://$(find delivery_robot_bringup)/meshes/castor.dae; visual mesh filename=file://$(find delivery_robot_bringup)/meshes/castor.dae
- link rr_castor_housing_link: geometry collision mesh filename=file://$(find delivery_robot_bringup)/meshes/castor_housing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; visual mesh filename=file://$(find delivery_robot_bringup)/meshes/castor_housing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
- link rr_castor_link: geometry collision mesh filename=file://$(find delivery_robot_bringup)/meshes/castor.dae; visual mesh filename=file://$(find delivery_robot_bringup)/meshes/castor.dae

File: src/delivery_robot_bringup/urdf/rover_4wd.urdf (robot description, URDF)
Before this commit: robot rover_4wd, 6 links, 5 joints
Links:
- link chassis_link: geometry collision mesh filename=file://$(find delivery_robot_bringup)/meshes/flipper_chassi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; collision mesh filename=file://$(find delivery_robot_bringup)/meshes/flipper_track.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
- link fl_wheel_link: geometry collision mesh filename=file://$(find delivery_robot_bringup)/meshes/pro_tire.dae; visual mesh filename=file://$(find delivery_robot_bringup)/meshes/pro_tire.dae
- link fr_wheel_link: geometry collision mesh filename=file://$(find delivery_robot_bringup)/meshes/pro_tire.dae; visual mesh filename=file://$(find delivery_robot_bringup)/meshes/pro_tire.dae
- link rl_wheel_link: geometry collision mesh filename=file://$(find delivery_robot_bringup)/meshes/pro_tire.dae; visual mesh filename=file://$(find delivery_robot_bringup)/meshes/pro_tire.dae
- link rr_wheel_link: geometry collision mesh filename=file://$(find delivery_robot_bringup)/meshes/pro_tire.dae; visual mesh filename=file://$(find delivery_robot_bringup)/meshes/pro_tire.dae
